Commit message: Fixed sensor_kit.xacro

File: f1tenth_sensor_kit_description/urdf/sensor_kit.xacro (robot description, xacro)
@@ -37,27 +37,27 @@
       </link>
     </xacro:macro>
-    <xacro:laser parent="sensor_kit_base_link" name="laser" namespace="">
-      <origin
-        xyz="${calibration['sensor_kit_base_link']['lidar']['x']}
-             ${calibration['sensor_kit_base_link']['lidar']['y']}
-             ${calibration['sensor_kit_base_link']['lidar']['z']}"
-        rpy="${calibration['sensor_kit_base_link']['lidar']['roll']}
-             ${calibration['sensor_kit_base_link']['lidar']['pitch']}
-             ${calibration['sensor_kit_base_link']['lidar']['yaw']}"
-      />
-    </xacro:laser>
+    <xacro:laser_macro
+            parent="sensor_kit_base_link"
+            x="${calibration['sensor_kit_base_link']['lidar']['x']}"
+            y="${calibration['sensor_kit_base_link']['lidar']['y']}"
+            z="${calibration['sensor_kit_base_link']['lidar']['z']}"
+            roll="${calibration['sensor_kit_base_link']['lidar']['roll']}"
+            pitch="${calibration['sensor_kit_base_link']['lidar']['pitch']}"
+            yaw="${calibration['sensor_kit_base_link']['lidar']['yaw']}"
+    />
     <!--  camera: Realsense D435i -->
-    <xacro:sensor_d435
+    <xacro:sensor_d435i
       name="camera"
       parent="sensor_kit_base_link"
-      use_nominal_extrinsics="$(arg use_nominal_extrinsics)"
-      namespace=""
-      x="${calibration['sensor_kit_base_link']['camera_link']['x']}"
-      y="${calibration['sensor_kit_base_link']['camera_link']['y']}"
-      z="${calibration['sensor_kit_base_link']['camera_link']['z']}"
-      roll="${calibration['sensor_kit_base_link']['camera_link']['roll']}"
-      pitch="${calibration['sensor_kit_base_link']['camera_link']['pitch']}"
-      yaw="${calibration['sensor_kit_base_link']['camera_link']['yaw']}"
-    />
+      use_nominal_extrinsics="$(arg use_nominal_extrinsics)">
+      <origin
+        xyz="${calibration['sensor_kit_base_link']['camera_link']['x']}
+             ${calibration['sensor_kit_base_link']['camera_link']['y']}
+             ${calibration['sensor_kit_base_link']['camera_link']['z']}"
+        rpy="${calibration['sensor_kit_base_link']['camera_link']['roll']}
+             ${calibration['sensor_kit_base_link']['camera_link']['pitch']}
+             ${calibration['sensor_kit_base_link']['camera_link']['yaw']}"
+      />
+    </xacro:sensor_d435i >
     <!-- imu -->
     <xacro:imu_macro

Commit message: Updated sensor extrinsic transformations to latest values.

File: f1tenth_sensor_kit_description/urdf/sensor_kit.xacro (robot description, xacro)
@@ -7,5 +7,5 @@
     <xacro:arg name="gpu" default="false"/>
     <xacro:arg name="config_dir" default="$(find f1tenth_sensor_kit_description)/config"/>
-    <xacro:arg name="use_nominal_extrinsics" default="False" /> <!-- Realsense nominal extrinsics -->
+    <xacro:arg name="use_nominal_extrinsics" default="False" /> <!-- Realsense nominal extrinsics. Use when simulating but disable with a real camera publishing calibrated extrinsics. -->
     <xacro:property name="sensor_kit_base_link" default="sensor_kit_base_link"/>
     <joint name="${sensor_kit_base_link}_joint" type="fixed">

File: f1tenth_sensor_kit_description/urdf/sensors.xacro (robot description, xacro)
@@ -17,3 +17,32 @@
     yaw="${calibration['base_link']['sensor_kit_base_link']['yaw']}"
   />
+  <!-- Rear axle -->
+  <xacro:macro name="static_tf_macro" params="parent child name x y z roll pitch yaw">
+    <joint name="${name}_joint" type="fixed">
+      <origin
+        xyz="${x}
+             ${y}
+             ${z}"
+        rpy="${roll}
+             ${pitch}
+             ${yaw}"
+      />
+      <parent link="${parent}"/>
+      <child link="${child}"/>
+    </joint>
+    <link name="${name}">
+      <origin rpy="0 0 0" xyz="0 0 0"/>
+    </link>
+  </xacro:macro>
+    <xacro:static_tf_macro
+      parent="base_link"
+      child=""
+      name=""
+      x="${calibration['base_link']['rear_axle_link']['x']}"
+      y="${calibration['base_link']['rear_axle_link']['y']}"
+      z="${calibration['base_link']['rear_axle_link']['z']}"
+      roll="${calibration['base_link']['rear_axle_link']['roll']}"
+      pitch="${calibration['base_link']['rear_axle_link']['pitch']}"
+      yaw="${calibration['base_link']['rear_axle_link']['yaw']}"
+    />
 </robot>
